File: schematic/main_v1/main_v1.kicad_pcb (KiCad board)
At the start: 4 copper layers, 100.3 x 100.3 mm, 135 parts, among them J1 JST_SH_4, J10 JST_SH_4, J2 JST_XH_4, J3 JST_XH_4, J4 JST_GH_6, J5 JST_XH_4, J6 JST_GH_6, J7 JST_XH_4, J8 JST_XH_4, J9 Conn_Coaxial, Q10 MMBT3904, Q11 MMBT3904, Q2 DMG2301L, Q3 PMN48XP, Q4 DMG2301L, Q5 DMG2301L, Q6 DMG2301L, Q7 DMG2301L, Q8 MMBT3904, Q9 PMN48XP, SW1 SW_DPST_x2, U1 Teensy4.1, U10 terminal-2, U11 BTN7030-1EPA, U12 BTN7030-1EPA, U13 BTN7030-1EPA, U14 BTN7030-1EPA, U15 NL17SZ17, U16 w25nxx, U17 SN65HVD230, U18 NL17SZ17, U19 NL17SZ17, U2 12v-engine, U20 NL17SZ17, U21 NL17SZ17, U22 NL17SZ17, U23 terminal-2, U24 terminal-2, U25 BTN7030-1EPA, U26 BTN7030-1EPA, U27 12v-in, U28 7v-in, U29 L7805, U3 12v-out, U30 Si7021-A20, U31 ltc2992, U32 RFM98W-433S2, U33 GY91, U35 drotek_10dof, U4 TXS0104E, U5 NL17SZ17, U6 sparkfun_H3LIS331DL, U7 terminal-2, U8 terminal-2, U9 terminal-2

Commit message: bajs
Parts:
- C16: value 330nF -> 330n
- C17: value 100nF -> 100n
- C2: value 100pF -> 100n
- C22, C9: value 100nf -> 100n
- R11, R12: value 400 -> 402
Connections:
- D9 pad 2: (no net) -> unconnected-(D9-Pad2)
- U1 pad 38: (no net) -> unconnected-(U1-Pad38)
- U1 pad 45: (no net) -> /BUZZ
- U1 pad 50: (no net) -> unconnected-(U1-Pad50)
- U1 pad 51: (no net) -> unconnected-(U1-Pad51)
- U1 pad 53: (no net) -> unconnected-(U1-Pad53)
- U1 pad 54: (no net) -> unconnected-(U1-Pad54)
- U1 pad 55: (no net) -> unconnected-(U1-Pad55)
- U1 pad 56: (no net) -> unconnected-(U1-Pad56)
- U1 pad 57: (no net) -> unconnected-(U1-Pad57)
- U1 pad 58: (no net) -> unconnected-(U1-Pad58)
- U1 pad 59: (no net) -> unconnected-(U1-Pad59)
- U1 pad 60: (no net) -> unconnected-(U1-Pad60)
- U1 pad 61: (no net) -> unconnected-(U1-Pad61)
- U1 pad 62: (no net) -> unconnected-(U1-Pad62)
- U1 pad 63: (no net) -> unconnected-(U1-Pad63)
- U1 pad 64: (no net) -> unconnected-(U1-Pad64)
- U1 pad 65: (no net) -> unconnected-(U1-Pad65)
- U1 pad 66: (no net) -> unconnected-(U1-Pad66)
- U1 pad 67: (no net) -> unconnected-(U1-Pad67)
- U11 pad 4: (no net) -> unconnected-(U11-Pad4)
- U12 pad 4: (no net) -> unconnected-(U12-Pad4)
- U13 pad 4: (no net) -> unconnected-(U13-Pad4)
- U14 pad 4: (no net) -> unconnected-(U14-Pad4)
- U17 pad 5: (no net) -> unconnected-(U17-Pad5)
- U25 pad 4: (no net) -> unconnected-(U25-Pad4)
- U26 pad 4: (no net) -> unconnected-(U26-Pad4)
- U30 pad 3: (no net) -> unconnected-(U30-Pad3)
- U30 pad 4: (no net) -> unconnected-(U30-Pad4)
- U31 pad 12: (no net) -> unconnected-(U31-Pad12)
- U31 pad 13: (no net) -> unconnected-(U31-Pad13)
- U31 pad 14: (no net) -> unconnected-(U31-Pad14)
- U31 pad 3: (no net) -> unconnected-(U31-Pad3)
- U31 pad 4: (no net) -> unconnected-(U31-Pad4)
- U32 pad 11: (no net) -> unconnected-(U32-Pad11)
- U32 pad 12: (no net) -> unconnected-(U32-Pad12)
- U32 pad 15: (no net) -> unconnected-(U32-Pad15)
- U32 pad 16: (no net) -> unconnected-(U32-Pad16)
- U32 pad 7: (no net) -> unconnected-(U32-Pad7)
- U33 pad 2: (no net) -> unconnected-(U33-Pad2)
- U33 pad 7: (no net) -> unconnected-(U33-Pad7)
- U33 pad 8: (no net) -> unconnected-(U33-Pad8)
- U35 pad 1: (no net) -> unconnected-(U35-Pad1)
- U35 pad 3: (no net) -> unconnected-(U35-Pad3)
- U35 pad 4: (no net) -> unconnected-(U35-Pad4)
- U4 pad 12: (no net) -> unconnected-(U4-Pad12)
- U4 pad 13: (no net) -> unconnected-(U4-Pad13)
- U4 pad 2: (no net) -> unconnected-(U4-Pad2)
- U4 pad 3: (no net) -> unconnected-(U4-Pad3)
- U6 pad 1: (no net) -> unconnected-(U6-Pad1)
- U6 pad 2: (no net) -> unconnected-(U6-Pad2)
- U6 pad 3: (no net) -> unconnected-(U6-Pad3)
- U6 pad 4: (no net) -> unconnected-(U6-Pad4)
Other:
- net class Default removed
- net class high-power removed
- net class power removed
